File: Eagle/BMS/battery_monitor_6803-2 -no_uno.sch (EAGLE design)
At the start: 127 parts, among them IC1 MIC2920A-5.0WS, J1 ARDUINO_R3_SHIELDNOLABELS, Q1 MOSFET-PCHANNELIRLML2244, Q10 IRF9530, Q11 MOSFET-PCHANNELIRLML2244, Q12 MOSFET-PCHANNELIRLML2244, Q13 MOSFET-PCHANNELIRLML2244, Q14 PMOS_AO4435, Q2 MOSFET-NCHANNELBSS138, Q3 MOSFET-PCHANNELIRLML2244, Q4 MOSFET-PCHANNELIRLML2244, Q5 MOSFET-PCHANNELIRLML2244, Q6 MOSFET-NCHANNELBSS138, Q7 MOSFET-NCHANNELBSS138, Q9 PMOS_AO4435, X1 USB-M26FTR

Commit message: Created 2 new revisions of BMS board and updated firmware.
Parts:
- A0, A1, A2, A3, C10, C11, C12, C13, C14, C15, C16, C17, C4, C5, C6, C7, C9, DZ1, DZ2, DZ3, DZ4, DZ5, DZ6, F1, IC1, J1, JP1, L1, LED1, LED2, LED3, LED4, LED5, LED6, LED7, LED8, Q1, Q10, Q11, Q12, Q13, Q14, Q2, Q3, Q4, Q5, Q6, Q7, Q9, R1, R10, R11, R12, R13, R14, R15, R16, R17, R18, R19, R2, R20, R21, R22, R23, R24, R25, R26, R28, R29, R3, R30, R31, R32, R33, R34, R35, R36, R37, R38, R39, R4, R40, R41, R42, R43, R44, R45, R5, R6, R7, R8, R9, SJ1, SJ2, SJ3, SJ4, SJ5, SJ6, SJ7, SJ8, TOS, U$1, U$10, U$11, U$12, U$13, U$14, U$15, U$16, U$17, U$2, U$3, U$4, U$5, U$6, U$7, U$8, U$9, X18: OC_NEWARK (none) -> unknown
- C1, C18, C19, C2, C20, C3: MPN (none) -> 0402ZD104KAT2A; OC_NEWARK (none) -> 96M1117
