File: Eagle/BMS/LTC6803 breakout.brd (EAGLE design)
At the start: 21.3 x 21.4 mm, 45 parts, among them P1 SINGLE_TERMINAL, P10 SINGLE_TERMINAL, P11 SINGLE_TERMINAL, P12 SINGLE_TERMINAL, P13 SINGLE_TERMINAL, P14 SINGLE_TERMINAL, P15 SINGLE_TERMINAL, P16 SINGLE_TERMINAL, P17 SINGLE_TERMINAL, P18 SINGLE_TERMINAL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

Commit message: Added new board order details.
Parts:
- renumbered P1 to V+, P10 to C8, P11 to S8, P12 to C7, P13 to S7, P14 to C6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
