File: Eagle/BMS/LTC6803 breakout.sch (EAGLE design)
At the start: 45 parts, among them P1 SINGLE_TERMINAL, P10 SINGLE_TERMINAL, P11 SINGLE_TERMINAL, P12 SINGLE_TERMINAL, P13 SINGLE_TERMINAL, P14 SINGLE_TERMINAL, P15 SINGLE_TERMINAL, P16 SINGLE_TERMINAL, P17 SINGLE_TERMINAL, P18 SINGLE_TERMINAL, P19 SINGLE_TERMINAL, P2 SINGLE_TERMINAL, P20 SINGLE_TERMINAL, P21 SINGLE_TERMINAL, P22 SINGLE_TERMINAL, P23 SINGLE_TERMINAL, P24 SINGLE_TERMINAL, P25 SINGLE_TERMINAL, P26 SINGLE_TERMINAL, P27 SINGLE_TERMINAL, P28 SINGLE_TERMINAL, P29 SINGLE_TERMINAL, P3 SINGLE_TERMINAL, P30 SINGLE_TERMINAL, P31 SINGLE_TERMINAL, P32 SINGLE_TERMINAL, P33 SINGLE_TERMINAL, P34 SINGLE_TERMINAL, P35 SINGLE_TERMINAL, P36 SINGLE_TERMINAL, P37 SINGLE_TERMINAL, P38 SINGLE_TERMINAL, P39 SINGLE_TERMINAL, P4 SINGLE_TERMINAL, P40 SINGLE_TERMINAL, P41 SINGLE_TERMINAL, P42 SINGLE_TERMINAL, P43 SINGLE_TERMINAL, P44 SINGLE_TERMINAL, P5 SINGLE_TERMINAL, P6 SINGLE_TERMINAL, P7 SINGLE_TERMINAL, P8 SINGLE_TERMINAL, P9 SINGLE_TERMINAL

Commit message: Finished new BMS boards in Eagle.
Parts:
- P1, P10, P11, P12, P13, P14, P15, P16, P17, P18, P19, P2, P20, P21, P22, P23, P24, P25, P26, P27, P28, P29, P3, P30, P31, P32, P33, P34, P35, P36, P37, P38, P39, P4, P40, P41, P42, P43, P44, P5, P6, P7, P8, P9, U$21: OC_NEWARK (none) -> unknown

Commit message: Added new board order details.
Parts:
- renumbered P1 to V+, P10 to C8, P11 to S8, P12 to C7, P13 to S7, P14 to C6, P15 to S6, P16 to C5, P17 to S5, P18 to C4, P19 to S4, P2 to C15, P20 to C3, P21 to S3, P22 to C2, P23 to S2, P24 to C1, P25 to S1, P26 to V-, P27 to NC, P28 to VTEMP1, P29 to VTEMP2, P3 to S12, P30 to VREF, P31 to VREG, P32 to TOS, P33 to NC1, P34 to WDTB, P35 to GPIO1, P36 to GPIO2, P37 to A0, P38 to A1, P39 to A2, P4 to C11, P40 to A3, P41 to SCKI, P42 to SDI, P43 to SDO, P44 to CSBI, P5 to S11, P6 to C10, P7 to S10, P8 to C9, P9 to S9
