File: Eagle/BMS/battery_monitor_6803-2_Rev3.brd (EAGLE design)
At the start: 65.8 x 53.3 mm, 66 parts, among them Q1 MOSFET-PCHANNELIRLML2244, Q10 IRF9530, Q2 MOSFET-NCHANNELBSS138, Q3 MOSFET-PCHANNELIRLML2244, Q4 MOSFET-PCHANNELIRLML2244, Q5 MOSFET-PCHANNELIRLML2244, Q6 MOSFET-NCHANNELBSS138, Q7 MOSFET-NCHANNELBSS138, Q8 MOSFET-NCHANNELBSS138, Q9 PMOS_AO4435

Commit message: Finished new BMS boards in Eagle.
Routing:
- net GND: vias 16 -> 15
Changed lines of the file:
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@@
 <via x="26.416" y="10.541" extent="1-16" drill="0.6"/>
 <wire x1="26.416" y1="10.541" x2="26.924" y2="10.541" width="0.2032" layer="16"/>
-<via x="3.048" y="8.763" extent="1-16" drill="0.6"/>
 <wire x1="15.367" y1="29.591" x2="11.342" y2="29.591" width="0.3048" layer="1"/>
 <wire x1="11.342" y1="29.591" x2="10.668" y2="30.265" width="0.3048" layer="1"/>

Commit message: Final revisions on BMS boards.
Changed lines of the file:
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@@
 <text x="8.509" y="20.574" size="0.508" layer="21">ESTOP1</text>
 <text x="8.509" y="17.907" size="0.508" layer="21">ESTOP2</text>
-<text x="9.779" y="13.843" size="0.508" layer="21" rot="R90">CHGR
-OUT</text>
 <text x="9.652" y="2.667" size="0.508" layer="21" rot="R90">CHGR
 OUT</text>

Commit message: Latest BMS Rev3 and Rev4 edits.
Routing:
- net CHARGER_IN: track 69.9 -> 63.9 mm
- net BATTERY+: track 16.2 -> 16.0 mm, vias 1 -> 0
Changed lines of the file:
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@@
 <wire x1="24.003" y1="5.461" x2="23.137" y2="5.461" width="0.2032" layer="1"/>
 <wire x1="23.137" y1="5.461" x2="23.071" y2="5.527" width="0.2032" layer="1"/>
-<wire x1="23.071" y1="5.527" x2="18.349" y2="5.527" width="0.2032" layer="1"/>
-<wire x1="18.349" y1="5.527" x2="13.716" y2="9.779" width="0.2032" layer="1"/>
-<wire x1="13.716" y1="9.779" x2="9.398" y2="7.493" width="0.2032" layer="1"/>
 <contactref element="R25" pad="2"/>
 <wire x1="35.521" y1="6.223" x2="35.521" y2="3.849" width="0.2032" layer="1"/>
@@
 <wire x1="22.352" y1="11.938" x2="21.59" y2="11.938" width="0.6096" layer="1"/>
 <wire x1="21.59" y1="11.938" x2="21.336" y2="12.192" width="0.6096" layer="1"/>
-<wire x1="4.953" y1="6.223" x2="9.398" y2="7.493" width="1.016" layer="1"/>
-<wire x1="9.398" y1="7.493" x2="13.716" y2="9.906" width="1.016" layer="1"/>
-<wire x1="13.716" y1="9.906" x2="20.955" y2="9.906" width="1.016" layer="1"/>
-<wire x1="20.955" y1="9.906" x2="21.082" y2="10.033" width="1.016" layer="1"/>
-<wire x1="21.082" y1="10.033" x2="21.082" y2="11.43" width="1.016" layer="1"/>
-<wire x1="21.082" y1="11.43" x2="21.59" y2="11.938" width="1.016" layer="1"/>
+<wire x1="15.367" y1="9.906" x2="15.113" y2="9.906" width="0.8128" layer="1"/>
+<wire x1="15.113" y1="9.906" x2="11.43" y2="6.223" width="0.8128" layer="1"/>
+<wire x1="11.43" y1="6.223" x2="4.953" y2="6.223" width="0.8128" layer="1"/>
+<wire x1="23.071" y1="5.527" x2="23.01" y2="5.588" width="0.2032" layer="1"/>
+<wire x1="23.01" y1="5.588" x2="18.034" y2="5.588" width="0.2032" layer="1"/>
+<wire x1="18.034" y1="5.588" x2="15.367" y2="8.255" width="0.2032" layer="1"/>
+<wire x1="15.367" y1="8.255" x2="15.367" y2="9.906" width="0.2032" layer="1"/>
+<wire x1="15.367" y1="9.906" x2="19.05" y2="9.906" width="0.8128" layer="1"/>
+<wire x1="19.05" y1="9.906" x2="21.082" y2="11.938" width="0.8128" layer="1"/>
 </signal>
 <signal name="N$24">
@@
 <wire x1="14.097" y1="18.796" x2="15.963" y2="18.796" width="0.6096" layer="1"/>
 <contactref element="U$4" pad="P$1"/>
-<wire x1="4.953" y1="11.303" x2="6.477" y2="11.43" width="0.8128" layer="1"/>
-<via x="6.477" y="11.43" extent="1-16" drill="0.6"/>
-<wire x1="6.477" y1="11.43" x2="12.827" y2="18.796" width="0.8128" layer="16"/>
-<wire x1="12.827" y1="18.796" x2="14.097" y2="18.796" width="0.8128" layer="16"/>
 <contactref element="R26" pad="2"/>
 <wire x1="17.272" y1="17.487" x2="15.963" y2="18.796" width="0.6096" layer="1"/>
+<wire x1="14.097" y1="18.796" x2="12.446" y2="18.796" width="0.8128" layer="16"/>
+<wire x1="12.446" y1="18.796" x2="4.953" y2="11.303" width="0.8128" layer="16"/>
 </signal>
 <signal name="ESTOP1">

Commit message: Encoder design Rev1 changes.
Parts:
- removed D2: PMLL41SOD80C, diode:SOD80C
Connections:
- removed net CHARGER_OUT: Q9.5, Q9.6, Q9.7, Q9.8, U$4.P$4
- net +12: now also U$4.P$4; no longer D2.C
- net BATTERY+: now also Q9.5, Q9.6, Q9.7, Q9.8
- net ESTOP2: no longer D2.A
Routing:
- net CHARGER_OUT: track 31.8 -> 0.00 mm, vias 1 -> 0
- net ESTOP2: track 55.2 -> 35.0 mm, vias 4 -> 1
- net +12: track 75.4 -> 89.9 mm
- net BATTERY+: track 16.0 -> 24.2 mm
Other:
- board text added: "VOUT"
- board text removed: "CHGR OUT"
Changed lines of the file:
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@@
 <text x="8.509" y="20.574" size="0.508" layer="21">ESTOP1</text>
 <text x="8.509" y="17.907" size="0.508" layer="21">ESTOP2</text>
-<text x="9.652" y="2.667" size="0.508" layer="21" rot="R90">CHGR
-OUT</text>
+<text x="9.017" y="2.794" size="0.508" layer="21" rot="R90">VOUT</text>
 </plain>
 <attributes>
@@
 <attribute name="MPN" value="CRCW06034K70FKEA" x="38.735" y="12.446" size="1.778" layer="27" rot="R180" display="off"/>
 </element>
-<element name="D2" library="diode" package="SOD80C" value="PMLL41SOD80C" x="6.35" y="41.021" smashed="yes" rot="R270">
-<attribute name="NAME" x="4.826" y="43.434" size="1.27" layer="25"/>
-<attribute name="OC_NEWARK" value="18C6408" x="6.35" y="41.021" size="1.778" layer="27" rot="R270" display="off"/>
-<attribute name="MF" value="FAIRCHILD SEMICONDUCTOR" x="6.35" y="41.021" size="1.778" layer="27" rot="R270" display="off"/>
-<attribute name="MPN" value="FDLL4148" x="6.35" y="41.021" size="1.778" layer="27" rot="R270" display="off"/>
-</element>
 <element name="I2C" library="isaac1" package="SCREW_TERMINAL_2" value="SCREW_TERMINAL_2" x="15.367" y="24.892" smashed="yes">
 <attribute name="OC_NEWARK" value="12H8386" x="15.367" y="24.892" size="1.778" layer="27" display="off"/>
@@
 <signal name="+12">
 <contactref element="U$8" pad="VIN"/>
-<contactref element="D2" pad="C"/>
 <wire x1="30.48" y1="51.562" x2="30.48" y2="51.943" width="0.4064" layer="1"/>
 <wire x1="30.48" y1="51.943" x2="29.21" y2="53.213" width="0.4064" layer="1"/>
@@
 <wire x1="2.667" y1="26.035" x2="2.667" y2="39.96441875" width="1.016" layer="1"/>
 <wire x1="2.667" y1="39.96441875" x2="2.8357" y2="40.13311875" width="1.016" layer="1"/>
-<wire x1="2.8357" y1="40.13311875" x2="6.35" y2="42.721" width="1.016" layer="1"/>
 <wire x1="12.230846875" y1="16.256" x2="2.667" y2="25.819846875" width="0.8128" layer="1"/>
 <wire x1="2.667" y1="25.819846875" x2="2.667" y2="26.035" width="0.8128" layer="1"/>
+<contactref element="U$4" pad="P$4"/>
+<wire x1="4.953" y1="3.683" x2="7.493" y2="3.683" width="0.8128" layer="16"/>
+<wire x1="7.493" y1="3.683" x2="9.525" y2="5.715" width="0.8128" layer="16"/>
+<wire x1="9.525" y1="5.715" x2="9.525" y2="13.550153125" width="0.8128" layer="16"/>
+<wire x1="9.525" y1="13.550153125" x2="12.230846875" y2="16.256" width="0.8128" layer="16"/>
+<wire x1="12.230846875" y1="16.256" x2="14.097" y2="16.256" width="0.8128" layer="16"/>
 </signal>
 <signal name="VREG">
@@
 <wire x1="24.638" y1="14.732" x2="23.876" y2="15.494" width="0.2032" layer="1"/>
 </signal>
-<signal name="CHARGER_OUT">
-<contactref element="Q9" pad="5"/>
-<contactref element="Q9" pad="6"/>
-<contactref element="Q9" pad="7"/>
-<contactref element="Q9" pad="8"/>
-<wire x1="20.066" y1="20.694" x2="21.336" y2="20.694" width="0.8128" layer="1"/>
-<wire x1="21.336" y1="20.694" x2="22.606" y2="20.694" width="0.8128" layer="1"/>
-<wire x1="22.606" y1="20.694" x2="23.876" y2="20.694" width="0.8128" layer="1"/>
-<contactref element="U$4" pad="P$4"/>
-<wire x1="20.066" y1="20.694" x2="18.923" y2="20.694" width="0.8128" layer="1"/>
-<wire x1="18.923" y1="20.694" x2="18.923" y2="11.43" width="0.8128" layer="1"/>
-<via x="18.923" y="11.43" extent="1-16" drill="0.6"/>
-<wire x1="18.923" y1="11.43" x2="18.923" y2="11.049" width="0.8128" layer="16"/>
-<wire x1="18.923" y1="11.049" x2="14.605" y2="6.731" width="0.8128" layer="16"/>
-<wire x1="14.605" y1="6.731" x2="11.938" y2="6.731" width="0.8128" layer="16"/>
-<wire x1="11.938" y1="6.731" x2="8.636" y2="3.429" width="0.8128" layer="16"/>
-<wire x1="8.636" y1="3.429" x2="5.207" y2="3.429" width="0.8128" layer="16"/>
-<wire x1="5.207" y1="3.429" x2="4.953" y2="3.683" width="0.8128" layer="16"/>
-</signal>
 <signal name="ESTOP2">
 <wire x1="33.02" y1="13.462" x2="31.115" y2="11.811" width="0.8128" layer="1"/>
 <via x="31.115" y="11.811" extent="1-16" drill="0.6"/>
-<wire x1="31.115" y1="11.811" x2="22.352" y2="11.684" width="0.8128" layer="16"/>
-<wire x1="22.352" y1="11.684" x2="19.1516" y2="15.4178" width="0.8128" layer="16"/>
-<wire x1="19.1516" y1="15.4178" x2="18.288" y2="18.796" width="0.8128" layer="16"/>
-<via x="14.605" y="20.525" extent="1-16" drill="0.6"/>
-<wire x1="14.605" y1="20.525" x2="16.559" y2="20.525" width="0.6096" layer="16"/>
-<wire x1="16.559" y1="20.525" x2="18.288" y2="18.796" width="0.6096" layer="16"/>
 <contactref element="U$6" pad="P$2"/>
-<via x="10.795" y="24.638" extent="1-16" drill="0.6"/>
-<wire x1="10.795" y1="24.638" x2="6.35" y2="29.083" width="0.6096" layer="16"/>
-<wire x1="6.35" y1="29.083" x2="6.35" y2="36.83" width="0.6096" layer="16"/>
-<via x="6.35" y="36.83" extent="1-16" drill="0.6"/>
 <wire x1="5.08" y1="18.288" x2="5.334" y2="18.542" width="0.6096" layer="16"/>
-<wire x1="5.334" y1="18.542" x2="10.6435" y2="24.4865" width="0.6096" layer="16"/>
-<wire x1="10.6435" y1="24.4865" x2="10.6435" y2="24.7895" width="0.6096" layer="16"/>
-<wire x1="10.6435" y1="24.7895" x2="10.795" y2="24.638" width="0.6096" layer="16"/>
-<wire x1="14.605" y1="20.525" x2="14.605" y2="20.828" width="0.6096" layer="1"/>
-<wire x1="14.605" y1="20.828" x2="10.795" y2="24.638" width="0.6096" layer="1"/>
-<contactref element="D2" pad="A"/>
 <contactref element="Q6" pad="3"/>
-<wire x1="6.35" y1="36.83" x2="6.35" y2="39.321" width="0.6096" layer="1"/>
+<wire x1="7.366" y1="20.574" x2="5.08" y2="18.288" width="0.8128" layer="16"/>
+<wire x1="31.115" y1="11.811" x2="22.606" y2="11.811" width="0.8128" layer="16"/>
+<wire x1="22.606" y1="11.811" x2="18.923" y2="15.494" width="0.8128" layer="16"/>
+<wire x1="18.923" y1="15.494" x2="18.923" y2="18.034" width="0.8128" layer="16"/>
+<wire x1="18.923" y1="18.034" x2="16.383" y2="20.574" width="0.8128" layer="16"/>
+<wire x1="16.383" y1="20.574" x2="7.366" y2="20.574" width="0.8128" layer="16"/>
 <wire x1="33.02" y1="13.462" x2="33.19" y2="13.462" width="0" layer="19" extent="1-1"/>
 </signal>
 <signal name="BATTERY+">
 <contactref element="Q10" pad="S"/>
-<wire x1="14.097" y1="18.796" x2="15.963" y2="18.796" width="0.6096" layer="1"/>
 <contactref element="U$4" pad="P$1"/>
 <contactref element="R26" pad="2"/>
-<wire x1="17.272" y1="17.487" x2="15.963" y2="18.796" width="0.6096" layer="1"/>
 <wire x1="14.097" y1="18.796" x2="12.446" y2="18.796" width="0.8128" layer="16"/>
 <wire x1="12.446" y1="18.796" x2="4.953" y2="11.303" width="0.8128" layer="16"/>
+<contactref element="Q9" pad="7"/>
+<contactref element="Q9" pad="5"/>
+<contactref element="Q9" pad="8"/>
+<contactref element="Q9" pad="6"/>
+<wire x1="23.876" y1="20.694" x2="22.606" y2="20.694" width="0.8128" layer="1"/>
+<wire x1="21.336" y1="20.694" x2="20.066" y2="20.694" width="0.8128" layer="1"/>
+<wire x1="22.606" y1="20.694" x2="21.336" y2="20.694" width="0.8128" layer="1"/>
+<wire x1="20.066" y1="20.694" x2="20.0491" y2="20.701" width="0.8128" layer="1" curve="45"/>
+<wire x1="20.0491" y1="20.701" x2="18.923" y2="20.701" width="0.8128" layer="1"/>
+<wire x1="18.923" y1="20.701" x2="17.4579875" y2="19.2359875" width="0.8128" layer="1"/>
+<wire x1="17.4579875" y1="19.2359875" x2="17.272" y2="18.786975" width="0.8128" layer="1" curve="45"/>
+<wire x1="17.272" y1="18.786975" x2="17.272" y2="17.487" width="0.8128" layer="1"/>
+<wire x1="14.097" y1="18.796" x2="14.1187875" y2="18.786975" width="0.8128" layer="1" curve="45"/>
+<wire x1="14.1187875" y1="18.786975" x2="17.272" y2="18.786975" width="0.8128" layer="1"/>
 </signal>
 <signal name="ESTOP1">
