File: Eagle/BMS/battery_monitor_6803-2_Rev6.sch (EAGLE design)
At the start: 68 parts, among them IC1 MIC2954-03WS, Q1 MOSFET-PCHANNELIRLML2244, Q10 IRF9530, Q2 MOSFET-NCHANNELBSS138, Q3 MOSFET-PCHANNELIRLML2244, Q4 MOSFET-PCHANNELIRLML2244, Q5 MOSFET-PCHANNELIRLML2244, Q6 MOSFET-NCHANNELBSS138, Q7 MOSFET-NCHANNELBSS138, Q8 MOSFET-NCHANNELBSS138, Q9 PMOS_AO4435

Commit message: Added voltage regulator to charging circuit of BMS.
Parts:
- removed A0: (no value), SparkFun:SOLDERJUMPER_2WAYS
- removed U$7: TACTILE-SWITCH-7914G, GeekAmmo:TACTILE-SWITCH-7914G
- removed U$8: ARDUINO_R3_SHIELD, SparkFun-Boards:ARDUINO_R3_SHIELD
- removed U$9: LTC6803, Clayton:LTC6803_BREAKOUT
- added A4: (no value), SparkFun:SOLDERJUMPER_2WAYS
- added D3: SMD26PL-TP, SparkFun-DiscreteSemi:DIODESOD123
- added U$5: RESISTOR-POWER-3W, isaac1:RESISTOR-POWER-3W
- added X1: W237-07P, con-wago-508:W237-07P
- C1: value 0.1uF -> 1uF; MF AVX CORPORATION -> (none); MPN 0603YG104ZAT2A -> C0603X5R0J105M030BC; OC_NEWARK 01H6821 -> 04X3184; PROD_ID (none) -> CAP-08390; VALUE (none) -> 0.1uF
- C4: value 1uF -> 0.1uF; MF (none) -> AVX CORPORATION; MPN C0603X5R0J105M030BC -> 0603YG104ZAT2A; OC_NEWARK 04X3184 -> 01H6821; PROD_ID CAP-08390 -> (none); VALUE 0.1uF -> (none)
- Q1, Q5: value MOSFET-PCHANNELIRLML2244 -> MOSFET-NCHANNELBSS138; device SparkFun-DiscreteSemi:MOSFET-PCHANNELIRLML2244 -> SparkFun-DiscreteSemi:MOSFET-NCHANNELBSS138; MPN IRLML2244TRPBF -> IRLML0030TRPBF; OC_NEWARK 40T7448 -> 52R2613
- Q10: value IRF9530 -> PMOS_AO4435; device Adams Chips:IRF9530 -> isaac1:PMOS_AO4435; MPN NTE2383 -> SI9407BDY-T1-GE3; OC_NEWARK 14T4215 -> 16P3885
- Q2: value MOSFET-NCHANNELBSS138 -> MOSFET-PCHANNELIRLML2244; device SparkFun-DiscreteSemi:MOSFET-NCHANNELBSS138 -> SparkFun-DiscreteSemi:MOSFET-PCHANNELIRLML2244; MPN IRLML0030TRPBF -> IRLML2244TRPBF; OC_NEWARK 52R2613 -> 40T7448
- Q7: value MOSFET-NCHANNELBSS138 -> IRF9530; device SparkFun-DiscreteSemi:MOSFET-NCHANNELBSS138 -> Adams Chips:IRF9530; MPN IRLML0030TRPBF -> NTE2383; OC_NEWARK 52R2613 -> 14T4215
- Q8: value MOSFET-NCHANNELBSS138 -> MOSFET-PCHANNELIRLML2244; device SparkFun-DiscreteSemi:MOSFET-NCHANNELBSS138 -> SparkFun-DiscreteSemi:MOSFET-PCHANNELIRLML2244; MPN IRLML0030TRPBF -> IRLML2244TRPBF; OC_NEWARK 52R2613 -> 40T7448; PROD_ID TRANS-00830 -> (none)
- Q9: value PMOS_AO4435 -> MOSFET-NCHANNELBSS138; device isaac1:PMOS_AO4435 -> SparkFun-DiscreteSemi:MOSFET-NCHANNELBSS138; MPN SI9407BDY-T1-GE3 -> IRLML0030TRPBF; OC_NEWARK 16P3885 -> 52R2613; PROD_ID (none) -> TRANS-00830
- R11: value 100k -> 4.7k; MF FARNELL -> VISHAY/DALE; MPN MC0063W06035100K -> CRCW06034K70FKEA; OC_NEWARK 39K0075 -> 52K8494
- R12: value 4.7k -> 100; MF VISHAY/DALE -> (none); MPN CRCW06034K70FKEA -> ERJ-1GNF1000C; OC_NEWARK 52K8494 -> 05X8794
- R14: value 4.7k -> 100k; MF VISHAY/DALE -> FARNELL; MPN CRCW06034K70FKEA -> MC0063W06035100K; OC_NEWARK 52K8494 -> 39K0075
- R18: value 470 -> 4.7k; MF (none) -> VISHAY/DALE; MPN ERJ-P03F4700V -> CRCW06034K70FKEA; OC_NEWARK 05X8640 -> 52K8494
- R19: value 4.7k -> 470; MF VISHAY/DALE -> (none); MPN CRCW06034K70FKEA -> ERJ-P03F4700V; OC_NEWARK 52K8494 -> 05X8640
- R21, R25: value 4.7k -> 1Meg; MF VISHAY/DALE -> (none); MPN CRCW06034K70FKEA -> ERJ-3EKF1004V; OC_NEWARK 52K8494 -> 64R5311
- R22: value 1Meg -> 4.7k; MF (none) -> VISHAY/DALE; MPN ERJ-3EKF1004V -> CRCW06034K70FKEA; OC_NEWARK 64R5311 -> 52K8494
- R24: PROD_ID RES-07851 -> (none)
- R26: value 1Meg -> 4.7k; MF (none) -> VISHAY/DALE; MPN ERJ-3EKF1004V -> CRCW06034K70FKEA; OC_NEWARK 64R5311 -> 52K8494; PROD_ID (none) -> RES-07851
- R3: value 3.3k -> 100; MF VISHAY/DALE -> (none); MPN CRCW06033K00FKEA -> ERJ-1GNF1000C; OC_NEWARK 52K8368 -> 05X8794
- R4: value 100 -> 3.3k; MF (none) -> VISHAY/DALE; MPN ERJ-1GNF1000C -> CRCW06033K00FKEA; OC_NEWARK 05X8794 -> 52K8368
- R5: value 100 -> 4.7k; MF (none) -> VISHAY/DALE; MPN ERJ-1GNF1000C -> CRCW06034K70FKEA; OC_NEWARK 05X8794 -> 52K8494
- U$2: value RESISTOR-POWER-3W -> TACTILE-SWITCH-7914G; device isaac1:RESISTOR-POWER-3W -> GeekAmmo:TACTILE-SWITCH-7914G; MF (none) -> BOURNS, INC.; MPN ERG-3SJ200 -> 7914G-1-000E; OC_NEWARK 52W7905 -> 05B2757
- U$4: value SCREW_TERMINAL_4 -> LTC6803; device isaac1:SCREW_TERMINAL_4 -> Clayton:LTC6803_BREAKOUT; MF TYCO ELECTRONICS -> (none); MPN 282834-4 -> LTC6803IG-2#PBF; OC_NEWARK 12H8388 -> 27T5837
- U$6: value SCREW_TERMINAL_2 -> ARDUINO_R3_SHIELD; device Isaac:SCREW_TERMINAL_2 -> SparkFun-Boards:ARDUINO_R3_SHIELD; MF TYCO ELECTRONICS -> (none); MPN 282834-2 -> (none); OC_NEWARK 12H8386 -> unknown
Connections:
- removed net 5VREG: IC1.VO, Q10.S, R26.2
- removed net VIN: D2.A, Q10.D, U$8.VIN
- removed net WIRE: D2.C, U$4.P$4
- new net 12VREG: D2.A, IC1.VO, U$6.VIN
- new net 12VUNREG: D3.A, IC1.VI, Q7.D
- new net N$15: D2.C, X1-4.KL
- new net N$16: D3.C, X1-5.KL
- net +5: now also Q9.D, R21.1, R22.2, R25.1, R9.2, U$6.5V; no longer Q8.D, R14.2, R21.2, R22.1, R24.1, U$8.5V
- net A0: now also A3.2, U$4.AO; no longer A0.2, U$9.AO
- net A1: now also U$4.A1; no longer U$9.A1
- net A2: now also A4.2, U$4.A2; no longer A2.2, U$9.A2
- net A3: now also A2.2, U$4.A3; no longer A3.2, U$9.A3
- net ALL_SYSTEMS_GO: now also R10.2, U$6.D8; no longer R13.2, U$8.D8
- net BATTERY+: now also Q7.S, R24.2, X1-1.KL; no longer IC1.VI, U$4.P$1
- net C1: now also C4.1, DZ3.C, R6.2, U$4.C1; no longer C3.1, DZ1.C, R4.2, U$9.C1
- net C12: now also R12.2, U$4.C10, U$4.C11, U$4.C12, U$4.C4, U$4.C5, U$4.C6, U$4.C7, U$4.C8, U$4.C9; no longer R7.2, U$9.C10, U$9.C11, U$9.C12, U$9.C4, U$9.C5, U$9.C6, U$9.C7, U$9.C8, U$9.C9
- net C2: now also C3.1, DZ1.A, R3.2, U$4.C2; no longer C2.1, DZ3.A, R5.2, U$9.C2
- net C3: now also C2.1, DZ1.C, R8.2, U$4.C3; no longer C1.1, DZ3.C, R6.2, U$9.C3
- net CHARGE: now also Q5.G, R13.2, U$6.*D9; no longer Q7.G, R12.2, U$8.*D9
- net CHARGER_CONNECTED: now also Q9.S, R18.2, U$6.D7; no longer Q8.S, R20.2, U$8.D7
- net CHARGER_IN: now also Q10.SOURCE, Q9.G, R20.2, R26.2, X1-3.KL; no longer Q8.G, Q9.SOURCE, R19.2, R25.2, U$4.P$3
- net ESTOP1: now also Q7.G, R24.1, U$2.3, U$2.4, X1-6.KL; no longer Q10.G, R26.1, U$6.P$1, U$7.3, U$7.4
- net ESTOP2: now also X1-7.KL; no longer U$6.P$2
- net GND: now also A4.3, DZ3.A, Q1.S, Q5.S, R18.1, R5.1, U$2.1, U$2.2, U$4.V-, U$6.GND@0, U$6.GND@1, U$6.GND@2, X1-2.KL; no longer A0.3, DZ1.A, Q2.S, Q7.S, R12.1, R19.1, U$4.P$2, U$7.1, U$7.2, U$8.GND@0, U$8.GND@1, U$8.GND@2, U$9.V-
- net GPIO1: now also U$4.GPIO1; no longer U$9.GPIO1
- net GPIO2: now also R21.2, U$4.GPIO2; no longer R22.2, U$9.GPIO2
- net MISO: now also R22.1, U$4.SDO, U$6.D12; no longer R21.1, U$8.D12, U$9.SDO
- net MOSI: now also U$4.SDI, U$6.*D11; no longer U$8.*D11, U$9.SDI
- net N$1: now also Q10.GATE, Q5.D, R26.1; no longer Q7.D, Q9.GATE, R25.1
- net N$10: now also Q3.D, U$3.P$1; no longer Q4.D, U$2.P$1
- net N$11: now also Q3.G; no longer Q4.G
- net N$12: now also Q8.D, R19.2, U$5.P$1; no longer Q5.D, R18.2, U$3.P$1
- net N$18: now also Q4.D, R7.2; no longer Q1.D, R8.2
- net N$2: now also Q2.S, R6.1, U$3.P$2; no longer Q3.S, R4.1, U$2.P$2
- net N$20: now also Q1.D, Q4.G, R11.1; no longer Q1.G, Q2.D, R9.1
- net N$23: now also R19.1; no longer R18.1
- net N$29: now also Q8.G, R4.1; no longer Q5.G, R3.1
- net N$3: now also Q3.S, R3.1, U$5.P$2; no longer Q4.S, R5.1, U$3.P$2
- net N$4: now also Q8.S, R12.1; no longer Q5.S, R6.1
- net N$5: now also Q2.D; no longer Q3.D
- net N$7: now also Q2.G; no longer Q3.G
- net N$8: now also Q10.DRAIN; no longer Q9.DRAIN
- net PWR: now also Q1.G, R5.2, U$6.*D6; no longer Q2.G, R10.2, U$8.*D6
- net S1: now also U$4.S1; no longer U$9.S1
- net S2: now also U$4.S2; no longer U$9.S2
- net S3: now also R4.2, U$4.S3; no longer R3.2, U$9.S3
- net SCK: now also U$4.SCKI, U$6.D13; no longer U$8.D13, U$9.SCKI
- net SCL: now also R9.1, U$6.SCL; no longer R15.1, U$8.SCL
- net SDA: now also R15.1, U$6.SDA; no longer R14.1, U$8.SDA
- net SS: now also U$4.CSBI, U$6.*D10; no longer U$8.*D10, U$9.CSBI
- net TOS: now also U$4.TOS; no longer U$9.TOS
- net V+: now also C6.2, Q4.S, R11.2, U$4.V+; no longer C5.2, Q1.S, R9.2, U$9.V+
- net VREF: now also C7.2, U$4.VREF; no longer C6.2, U$9.VREF
- net VREG: now also A4.1, C1.1, R14.2, U$4.VREG; no longer A0.1, C4.1, R11.2, U$9.VREG
- net VTEMP1: now also C5.2, R14.1, U$4.VTEMP1; no longer C7.2, R11.1, U$9.VTEMP1
- net WDTB: now also R25.2, U$4.WDTB; no longer R24.2, U$9.WDTB
Other:
- moved on the sheet: A2, A3, C1, C2, C3, C4, C5, C6, C7, D2, DZ1, DZ3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

Commit message: Changed linear regulator device.
Parts:
- IC1: value MIC2954-03WS -> MIC2920A-12WS
Changed lines of the file:
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@@
 </part>
 <part name="D1" library="SparkFun-DiscreteSemi" deviceset="DIODE" device="SOD123" value="SMD26PL-TP"/>
-<part name="IC1" library="linear" deviceset="MCP1703" device="DB" value="MIC2954-03WS"/>
+<part name="IC1" library="linear" deviceset="MCP1703" device="DB" value="MIC2920A-12WS"/>
 <part name="SUPPLY20" library="supply2" deviceset="GND" device=""/>
 <part name="X1" library="con-wago-508" deviceset="W237-07P" device="" value="W237-07P"/>
