File: Eagle/BMS/battery_monitor_6803-2_Rev2.sch (EAGLE design)
At the start: 65 parts, among them Q1 MOSFET-PCHANNELIRLML2244, Q10 IRF9530, Q2 MOSFET-NCHANNELBSS138, Q3 MOSFET-PCHANNELIRLML2244, Q4 MOSFET-PCHANNELIRLML2244, Q5 MOSFET-PCHANNELIRLML2244, Q6 MOSFET-NCHANNELBSS138, Q7 MOSFET-NCHANNELBSS138, Q8 MOSFET-NCHANNELBSS138, Q9 PMOS_AO4435

Commit message: Renumbered BMS revisions and wrote code for interrupt-driven encoders.
Parts:
- removed U$9: LTC6803, Clayton:LTC6803_BREAKOUT
- added U$5: LTC6803-2, isaac1:LTC6803-2
- Q1, Q3, Q4, Q5: MPN IRLML2244TRPBF -> SI2369DS-T1-GE3; OC_NEWARK 40T7448 -> 40X8697
- R26: value 1Meg -> 1MEG
Connections:
- removed net A0: A0.2, U$9.AO
- removed net A1: A1.2, U$9.A1
- removed net A2: A2.2, U$9.A2
- removed net A3: A3.2, U$9.A3
- removed net C1: C3.1, DZ1.C, DZ2.A, R4.2, U$9.C1
- removed net C12: R7.2, U$9.C10, U$9.C11, U$9.C12, U$9.C4, U$9.C5, U$9.C6, U$9.C7, U$9.C8, U$9.C9
- removed net C2: C2.1, DZ2.C, DZ3.A, R5.2, U$9.C2
- removed net C3: C1.1, DZ3.C, R6.2, U$9.C3
- removed net CHARGER_OUT: Q9.DRAIN, U$4.P$4
- removed net GPIO1: R23.2, U$9.GPIO1
- removed net GPIO2: R22.2, U$9.GPIO2
- removed net S1: R1.2, U$9.S1
- removed net S2: R2.2, U$9.S2
- removed net S3: R3.2, U$9.S3
- removed net TOS: TOS.2, U$9.TOS
- removed net V+: C5.2, Q1.S, R9.2, U$9.V+
- removed net VREF: C6.2, U$9.VREF
- removed net VTEMP1: C7.2, R11.1, THERM.P$1, U$9.VTEMP1
- removed net WDTB: R24.2, U$9.WDTB
- new net N$14: C1.1, DZ3.C, R6.2, U$5.C3
- new net N$15: C3.1, DZ1.C, DZ2.A, R4.2, U$5.C1
- new net N$16: C2.1, DZ2.C, DZ3.A, R5.2, U$5.C2
- new net N$17: R7.2, U$5.C10, U$5.C11, U$5.C12, U$5.C4, U$5.C5, U$5.C6, U$5.C7, U$5.C8, U$5.C9
- new net N$19: C5.2, Q1.S, R9.2, U$5.V+
- new net N$21: C7.2, R11.1, THERM.P$1, U$5.VTEMP1
- new net N$24: R22.2, U$5.GPIO2
- new net N$25: R23.2, U$5.GPIO1
- new net N$27: R24.2, U$5.WDTB
- new net N$28: A3.2, U$5.A3
- new net N$30: A2.2, U$5.A2
- new net N$31: A1.2, U$5.A1
- new net N$32: A0.2, U$5.AO
- new net N$33: TOS.2, U$5.TOS
- new net N$34: C6.2, U$5.VREF
- new net N$6: R2.2, U$5.S2
- new net N$8: R1.2, U$5.S1
- new net N$9: R3.2, U$5.S3
- net +12: now also U$4.P$4
- net BATTERY+: now also Q9.DRAIN
- net GND: now also U$5.V-; no longer U$9.V-
- net MISO: now also U$5.SDO; no longer U$9.SDO
- net MOSI: now also U$5.SDI; no longer U$9.SDI
- net SCK: now also U$5.SCKI; no longer U$9.SCKI
- net SS: now also U$5.CSBI; no longer U$9.CSBI
- net VREG: now also U$5.VREG; no longer U$9.VREG
Other:
- moved on the sheet: C6
