File: Eagle/Encoders/mag_encoder_Rev2.brd (EAGLE design)
At the start: 20 x 31.8 mm, 6 parts, among them IC1 A1203LH

Commit message: Mike maybe fixed his messup...
Parts:
- removed U$3: MOUNTING_SCREW-3MM, Clayton:MOUNTING_SCREW-3MM
Other:
- board size 20 x 31.8 mm -> 20 x 28.2 mm
Changed lines of the file:
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@@
 <?xml version="1.0" encoding="utf-8"?>
 <!DOCTYPE eagle SYSTEM "eagle.dtd">
-<eagle version="7.3.0">
+<eagle version="7.4.0">
 <drawing>
 <settings>
@@
 <text x="8.838" y="18.705" size="0.762" layer="25">VCC</text>
 <wire x1="4.75" y1="1.5" x2="4.75" y2="19.75" width="0" layer="20"/>
-<wire x1="19.75" y1="31" x2="19.75" y2="28.75" width="0" layer="20"/>
-<wire x1="-0.25" y1="31" x2="-0.25" y2="28.75" width="0" layer="20"/>
 <wire x1="14.75" y1="19.75" x2="14.75" y2="1.5" width="0" layer="20"/>
-<wire x1="2" y1="33.25" x2="17.5" y2="33.25" width="0" layer="20"/>
-<wire x1="19.75" y1="22" x2="19.75" y2="25.75" width="0" layer="20"/>
-<wire x1="-0.25" y1="22" x2="-0.25" y2="25.75" width="0" layer="20"/>
 <wire x1="14.75" y1="19.75" x2="17.5" y2="19.75" width="0" layer="20"/>
 <wire x1="4.75" y1="19.75" x2="2" y2="19.75" width="0" layer="20"/>
@@
 <wire x1="17.5" y1="19.75" x2="19.75" y2="22" width="0" layer="20"/>
 <wire x1="2" y1="19.75" x2="-0.25" y2="22" width="0" layer="20"/>
-<wire x1="19.75" y1="25.75" x2="14.75" y2="25.75" width="0" layer="20"/>
-<wire x1="14.75" y1="28.75" x2="19.75" y2="28.75" width="0" layer="20"/>
-<wire x1="14.75" y1="25.75" x2="14.75" y2="28.75" width="0" layer="20"/>
-<wire x1="-0.25" y1="25.75" x2="4.75" y2="25.75" width="0" layer="20"/>
-<wire x1="-0.25" y1="28.75" x2="4.75" y2="28.75" width="0" layer="20"/>
-<wire x1="4.75" y1="25.75" x2="4.75" y2="28.75" width="0" layer="20"/>
-<dimension x1="19.75" y1="28.75" x2="19.75" y2="25.75" x3="22.5" y3="27.25" textsize="1.778" layer="49" dtype="vertical"/>
-<dimension x1="-0.25" y1="25.75" x2="-0.25" y2="19.75" x3="-2.5" y3="22.75" textsize="1.778" layer="49" dtype="vertical"/>
-<dimension x1="-0.25" y1="28.75" x2="-0.25" y2="33.25" x3="-6.75" y3="31" textsize="1.778" layer="49" dtype="vertical"/>
-<dimension x1="17.5" y1="19.75" x2="17.25" y2="4.75" x3="19.75" y3="12.25" textsize="1.778" layer="49" dtype="vertical"/>
-<wire x1="19.75" y1="31" x2="17.5" y2="33.25" width="0" layer="20"/>
-<wire x1="2" y1="33.25" x2="-0.25" y2="31" width="0" layer="20"/>
+<wire x1="17.5" y1="29.75" x2="2" y2="29.75" width="0" layer="20"/>
+<wire x1="2" y1="29.75" x2="-0.25" y2="27.5" width="0" layer="20"/>
+<wire x1="17.5" y1="29.75" x2="19.75" y2="27.5" width="0" layer="20"/>
+<wire x1="19.75" y1="27.5" x2="19.75" y2="26" width="0" layer="20"/>
+<wire x1="19.75" y1="26" x2="14.75" y2="26" width="0" layer="20"/>
+<wire x1="19.75" y1="23.5" x2="19.75" y2="22" width="0" layer="20"/>
+<wire x1="19.75" y1="23.5" x2="14.75" y2="23.5" width="0" layer="20"/>
+<wire x1="14.75" y1="23.5" x2="14.75" y2="26" width="0" layer="20"/>
+<wire x1="-0.25" y1="23.5" x2="-0.25" y2="22" width="0" layer="20"/>
+<wire x1="4.75" y1="23.5" x2="-0.25" y2="23.5" width="0" layer="20"/>
+<wire x1="4.75" y1="23.5" x2="4.75" y2="26" width="0" layer="20"/>
+<wire x1="4.75" y1="26" x2="-0.25" y2="26" width="0" layer="20"/>
+<wire x1="-0.25" y1="27.5" x2="-0.25" y2="26" width="0" layer="20"/>
 </plain>
 <attributes>
@@
 </element>
 <element name="U$1" library="Clayton" package="3_PIN_JST-XH" value="3_PIN_JST-XH" x="14.7435" y="25.4995" rot="R180"/>
-<element name="U$3" library="Clayton" package="MOUNTING_SCREW-3MM" value="MOUNTING_SCREW-3MM" x="9.75" y="29.25"/>
 </elements>
 <signals>
