File: Eagle/Encoders/mag_encoder_Rev2.sch (EAGLE design)
At the start: 6 parts, among them IC1 A1203LH

Commit message: Mike maybe fixed his messup...
Parts:
- removed U$3: MOUNTING_SCREW-3MM, Clayton:MOUNTING_SCREW-3MM
Changed lines of the file:
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@@
 <?xml version="1.0" encoding="utf-8"?>
 <!DOCTYPE eagle SYSTEM "eagle.dtd">
-<eagle version="7.3.0">
+<eagle version="7.4.0">
 <drawing>
 <settings>
@@
 <part name="U$1" library="Clayton" deviceset="3_PIN_JST-XH" device=""/>
 <part name="SUPPLY4" library="supply2" deviceset="GND" device=""/>
-<part name="U$3" library="Clayton" deviceset="MOUNTING_SCREW-3MM" device=""/>
 </parts>
 <sheets>
@@
 <instance part="U$1" gate="G$1" x="91.44" y="66.04" rot="R270"/>
 <instance part="SUPPLY4" gate="GND" x="83.82" y="38.1"/>
-<instance part="U$3" gate="G$1" x="91.44" y="86.36"/>
 </instances>
 <busses>
